File: pcb/pixoclock.kicad_pcb (KiCad board)
At the start: 2 copper layers, 40 x 40 mm, 149 parts, among them SW1 Button, U1 STM32L072CBTx, Y1 32.768

Commit message: re-route all
Parts:
- added TP7: TestPoint, TestPoint:TestPoint_Pad_D1.0mm, B.Cu at (106.5, 109.2)
- moved TP4 3.68 mm to (94.5, 99.1)
- moved TP1 3.10 mm to (91.8, 102.0)
- moved TP2 3.10 mm to (91.8, 104.0)
- moved TP5 2.78 mm to (105.9, 94.1)
- moved TP6 2.40 mm to (108.4, 94.4)
- moved SW1 1.80 mm to (110.5, 99.7)
- moved Y1 0.50 mm to (107.1, 101.0)
Routing:
- net /CH6: track 59.7 -> 18.1 mm, vias 20 -> 11
- net /CH4: track 49.2 -> 13.7 mm, vias 19 -> 7
- net /CH5: track 53.2 -> 23.0 mm, vias 19 -> 6
- net /CH10: track 56.1 -> 29.3 mm, vias 18 -> 8
- net /CH11: track 51.3 -> 34.3 mm, vias 18 -> 8
- net /CH1: track 56.7 -> 43.8 mm, vias 20 -> 14
- net /NRST: track 0.00 -> 9.35 mm, vias 0 -> 2
- net /CH3: track 41.6 -> 32.9 mm, vias 22 -> 16
- net GND: track 53.7 -> 45.9 mm
- net /CH7: track 40.3 -> 33.0 mm, vias 22 -> 13
- net /CH12: track 40.8 -> 36.5 mm, vias 19 -> 9
- net +3V3: track 54.3 -> 50.7 mm
- net /CH9: track 42.2 -> 45.8 mm, vias 20 -> 11
- net /USB+: track 7.47 -> 4.37 mm
- net /USB-: track 7.47 -> 4.37 mm
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Other:
- board text added: "3V3"
- board text added: "CLK"
- board text added: "DIO"
- board text added: "GND"
- board text added: "RST"
- board text added: "USB+"
- board text added: "USB-"

Commit message: rerauted all for cheaper price
Routing:
- net /CH11: track 34.3 -> 91.2 mm, vias 8 -> 19
- net /CH10: track 29.3 -> 84.5 mm, vias 8 -> 20
- net /CH5: track 23.0 -> 72.0 mm, vias 6 -> 16
- net /CH4: track 13.7 -> 59.3 mm, vias 7 -> 19
- net /CH12: track 36.5 -> 81.0 mm, vias 9 -> 16
- net /CH2: track 44.8 -> 78.2 mm, vias 11 -> 16
- net /CH1: track 43.8 -> 75.8 mm, vias 14 -> 18
- net /CH6: track 18.1 -> 49.7 mm, vias 11 -> 18
- net /CH9: track 45.8 -> 73.3 mm, vias 11 -> 16
- net /CH3: track 32.9 -> 57.5 mm, vias 16 -> 21
- net /CH7: track 33.0 -> 53.1 mm, vias 13 -> 17
- net /CH8: track 37.6 -> 56.0 mm, vias 15 -> 18
- net GND: track 45.9 -> 45.7 mm, vias 3 -> 4
Other:
- board size 40 x 40 mm -> 40.2 x 40.2 mm
- board text added: "Made By: github.com/samux6146"
